File: 001.sch (EAGLE design)
At the start: 16 parts, among them IC1 74HC148N

Commit message: PCB パターンそれなりに完成
Other:
- note added: "8to3 Encoding Eva Board for Larning"
- note added: "HLED0001"
Changed lines of the file:
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@@
 <sheet>
 <plain>
+<text x="218.44" y="20.32" size="2.54" layer="91">HLED0001</text>
+<text x="162.56" y="7.62" size="3.81" layer="91">8to3 Encoding
+Eva Board for Larning</text>
 </plain>
 <instances>
@@
 </drawing>
 <compatibility>
+<note version="6.3" minversion="6.2.2" severity="warning">
+Since Version 6.2.2 text objects can contain more than one line,
+which will not be processed correctly with this version.
+</note>
 <note version="8.2" severity="warning">
 Since Version 8.2, EAGLE supports online libraries. The ids
